File: pcb/swaw_project.kicad_pcb (KiCad board)
At the start: 2 copper layers, 68.6 x 53.3 mm, 25 parts, among them P1 Power, P2 Analog, P3 Digital, P4 Digital, P5 CONN_01X01, P6 CONN_01X01, P7 CONN_01X01, P8 CONN_01X01, Q1 2N7002, Q2 2N7002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

Commit message: Changed some resistors to be normal size
Parts:
- R1, R2, R5, R6: footprint Resistor_SMD:R_0612_1632Metric_Pad1.18x3.40mm_HandSolder -> Resistor_SMD:R_0805_2012Metric_Pad1.15x1.40mm_HandSolder
- moved Q1 3.81 mm to (135.1, 92.1)
- moved Q2 3.81 mm to (126.2, 92.1)
Routing:
- net +3V3: track 90.4 -> 83.6 mm
- net /A5(SCL): track 14.2 -> 18.1 mm
- net /A4(SDA): track 12.9 -> 16.7 mm
- net Net-(Q1-Pad2): track 18.4 -> 14.7 mm
- net Net-(Q2-Pad2): track 19.2 -> 16.0 mm
