File: pcb/swaw_project.sch (KiCad schematic (older format))
At the start: 25 parts, among them P1 Power, P2 Analog, P3 Digital, P4 Digital, P5 CONN_01X01, P6 CONN_01X01, P7 CONN_01X01, P8 CONN_01X01, Q1 2N7002, Q2 2N7002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

Commit message: Changed some resistors to be normal size
Parts:
- R1, R2, R5, R6: footprint Resistor_SMD:R_0612_1632Metric_Pad1.18x3.40mm_HandSolder -> Resistor_SMD:R_0805_2012Metric_Pad1.15x1.40mm_HandSolder
Changed lines of the file:
@@
 F 0 "R2" H 5670 1346 50  0000 L CNN
 F 1 "10kΩ" H 5670 1255 50  0000 L CNN
-F 2 "Resistor_SMD:R_0612_1632Metric_Pad1.18x3.40mm_HandSolder" V 5530 1300 50  0001 C CNN
+F 2 "Resistor_SMD:R_0805_2012Metric_Pad1.15x1.40mm_HandSolder" V 5530 1300 50  0001 C CNN
 F 3 "~" H 5600 1300 50  0001 C CNN
 	1    5600 1300
@@
 F 0 "R1" H 5320 1346 50  0000 L CNN
 F 1 "10kΩ" H 5320 1255 50  0000 L CNN
-F 2 "Resistor_SMD:R_0612_1632Metric_Pad1.18x3.40mm_HandSolder" V 5180 1300 50  0001 C CNN
+F 2 "Resistor_SMD:R_0805_2012Metric_Pad1.15x1.40mm_HandSolder" V 5180 1300 50  0001 C CNN
 F 3 "~" H 5250 1300 50  0001 C CNN
 	1    5250 1300
@@
 F 0 "R5" H 6720 1546 50  0000 L CNN
 F 1 "10kΩ" H 6720 1455 50  0000 L CNN
-F 2 "Resistor_SMD:R_0612_1632Metric_Pad1.18x3.40mm_HandSolder" V 6580 1500 50  0001 C CNN
+F 2 "Resistor_SMD:R_0805_2012Metric_Pad1.15x1.40mm_HandSolder" V 6580 1500 50  0001 C CNN
 F 3 "~" H 6650 1500 50  0001 C CNN
 	1    6650 1500
@@
 F 0 "R6" H 7070 2046 50  0000 L CNN
 F 1 "10kΩ" H 7070 1955 50  0000 L CNN
-F 2 "Resistor_SMD:R_0612_1632Metric_Pad1.18x3.40mm_HandSolder" V 6930 2000 50  0001 C CNN
+F 2 "Resistor_SMD:R_0805_2012Metric_Pad1.15x1.40mm_HandSolder" V 6930 2000 50  0001 C CNN
 F 3 "~" H 7000 2000 50  0001 C CNN
 	1    7000 2000
